File: power-supply.kicad_pcb (KiCad board)
At the start: 2 copper layers, 11 parts, among them P1 CONN_01X02, P2 CONN_01X02, P3 CONN_01X03, U1 CONN_01X06

Commit message: added board
Parts:
- added REF**: 1pin, Connect:1pin, F.Cu at (91.4, 68.6)
- added REF**: 1pin, Connect:1pin, F.Cu at (113.0, 68.6)
- added REF**: 1pin, Connect:1pin, F.Cu at (91.4, 96.5)
- added REF**: 1pin, Connect:1pin, F.Cu at (113.0, 96.5)
- C1, C2, C3, C4, C5, JP1: moved to B.Cu
- moved C5 79.8 mm to (91.4, 87.6)
- moved C4 78.9 mm to (94.0, 91.4)
- moved P2 61.1 mm to (97.8, 69.8)
- moved P3 57.3 mm to (101.6, 95.2), turned to 180 degrees
- moved JP1 47.9 mm to (91.4, 74.9), turned to 270 degrees
- moved D1 39.9 mm to (101.6, 74.9)
- moved C3 37.4 mm to (111.8, 82.5)
- moved C1 30.6 mm to (111.8, 74.9)
- moved C2 30.5 mm to (108.0, 87.6)
- moved P1 26.7 mm to (106.7, 69.8)
- moved U1 20.4 mm to (96.5, 80.0)
Routing:
- net Net-(D1-Pad2): track 0.00 -> 19.4 mm
- net Net-(C4-Pad2): track 0.00 -> 17.9 mm
- net Net-(P3-Pad1): track 0.00 -> 17.9 mm
- net Net-(C1-Pad1): track 0.00 -> 11.0 mm

Commit message: final version
Parts:
- moved C3 4.02 mm to (108.0, 83.8)
- moved JP1 1.27 mm to (92.7, 74.9), turned to 90 degrees
Connections:
- C3 pad 1: Net-(C3-Pad1) -> Net-(C2-Pad1)
- P3 pad 1: Net-(P3-Pad1) -> Net-(C2-Pad1)
- U1 pad 4: Net-(P3-Pad1) -> Net-(C2-Pad1)
Routing:
- net Net-(C2-Pad1): track 0.00 -> 31.1 mm
- net Net-(C1-Pad1): track 11.0 -> 38.7 mm
- net Net-(P3-Pad1): track 17.9 -> 0.00 mm
- net Net-(JP1-Pad2): track 0.00 -> 6.88 mm
- net Net-(C4-Pad2): track 17.9 -> 24.5 mm
- added copper zone on B.Cu, net GND
